File: Titan67j60/Titan67j60_AnalogIN.sch (KiCad schematic (older format))
At the start: 71 parts, among them J10 Termistor 10k, J11 Termistor 10k, J12 Termistor 10k, J13 Termistor 10k, J14 Termistor 10k, J15 Termistor 10k, J16 Termistor 10k, J17 Termistor 10k, J32 CONN_01X03, J33 CONN_01X03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

Commit message: Работает минимальный набор до прикручивания TCP IP
Signed-off-by: Lehman3065 <lehman3065@gmail.com>
Parts:
- J10: value Termistor 10k -> Switch0
- J11: value Termistor 10k -> Switch1
- J12: value Termistor 10k -> Switch2
- J13: value Termistor 10k -> Switch3
- J14: value Termistor 10k -> Switch4
- J15: value Termistor 10k -> Switch5
- J16: value Termistor 10k -> Switch6
- J17: value Termistor 10k -> Switch7
- R39, R40, R41, R42, R43, R44, R45, R46: value 39k -> 10k
Connections:
- net +24V: no longer C16.1, R39.2, R40.2, R41.2, R42.2, R43.2, R44.2, R45.2, R46.2
- net +3V3: now also C16.1, R39.2, R40.2, R41.2, R42.2, R43.2, R44.2, R45.2, R46.2
Other:
- moved on the sheet: C16
Changed lines of the file:
@@
 P 6650 1600
 F 0 "J10" H 6850 1650 50  0000 C CNN
-F 1 "Termistor 10k" H 7000 1550 50  0000 C CNN
+F 1 "Switch0" H 7000 1550 50  0000 C CNN
 F 2 "Connectors_Phoenix:PhoenixContact_MC-G_02x5.08mm_Angled" H 6650 1600 50  0001 C CNN
 F 3 "" H 6650 1600 50  0001 C CNN
@@
 P 6650 1850
 F 0 "J11" H 6850 1900 50  0000 C CNN
-F 1 "Termistor 10k" H 7000 1800 50  0000 C CNN
+F 1 "Switch1" H 7000 1800 50  0000 C CNN
 F 2 "Connectors_Phoenix:PhoenixContact_MC-G_02x5.08mm_Angled" H 6650 1850 50  0001 C CNN
 F 3 "" H 6650 1850 50  0001 C CNN
@@
 P 6650 2100
 F 0 "J12" H 6850 2150 50  0000 C CNN
-F 1 "Termistor 10k" H 7000 2050 50  0000 C CNN
+F 1 "Switch2" H 7000 2050 50  0000 C CNN
 F 2 "Connectors_Phoenix:PhoenixContact_MC-G_02x5.08mm_Angled" H 6650 2100 50  0001 C CNN
 F 3 "" H 6650 2100 50  0001 C CNN
@@
 P 6650 2350
 F 0 "J13" H 6850 2400 50  0000 C CNN
-F 1 "Termistor 10k" H 7000 2300 50  0000 C CNN
+F 1 "Switch3" H 7000 2300 50  0000 C CNN
 F 2 "Connectors_Phoenix:PhoenixContact_MC-G_02x5.08mm_Angled" H 6650 2350 50  0001 C CNN
 F 3 "" H 6650 2350 50  0001 C CNN
@@
 P 6650 2600
 F 0 "J14" H 6850 2650 50  0000 C CNN
-F 1 "Termistor 10k" H 7000 2550 50  0000 C CNN
+F 1 "Switch4" H 7000 2550 50  0000 C CNN
 F 2 "Connectors_Phoenix:PhoenixContact_MC-G_02x5.08mm_Angled" H 6650 2600 50  0001 C CNN
 F 3 "" H 6650 2600 50  0001 C CNN
@@
 P 6650 2850
 F 0 "J15" H 6850 2900 50  0000 C CNN
-F 1 "Termistor 10k" H 7000 2800 50  0000 C CNN
+F 1 "Switch5" H 7000 2800 50  0000 C CNN
 F 2 "Connectors_Phoenix:PhoenixContact_MC-G_02x5.08mm_Angled" H 6650 2850 50  0001 C CNN
 F 3 "" H 6650 2850 50  0001 C CNN
@@
 P 6650 3100
 F 0 "J16" H 6850 3150 50  0000 C CNN
-F 1 "Termistor 10k" H 7000 3050 50  0000 C CNN
+F 1 "Switch6" H 7000 3050 50  0000 C CNN
 F 2 "Connectors_Phoenix:PhoenixContact_MC-G_02x5.08mm_Angled" H 6650 3100 50  0001 C CNN
 F 3 "" H 6650 3100 50  0001 C CNN
@@
 P 6650 3350
 F 0 "J17" H 6850 3400 50  0000 C CNN
-F 1 "Termistor 10k" H 7000 3300 50  0000 C CNN
+F 1 "Switch7" H 7000 3300 50  0000 C CNN
 F 2 "Connectors_Phoenix:PhoenixContact_MC-G_02x5.08mm_Angled" H 6650 3350 50  0001 C CNN
 F 3 "" H 6650 3350 50  0001 C CNN
@@
 P 8700 1550
 F 0 "R39" V 8750 1700 50  0000 L CNN
-F 1 "39k" V 8750 1300 50  0000 L CNN
+F 1 "10k" V 8750 1300 50  0000 L CNN
 F 2 "Resistors_SMD:R_0805" H 8700 1550 50  0001 C CNN
 F 3 "" H 8700 1550 50  0001 C CNN
@@
 P 8700 1800
 F 0 "R40" V 8750 1950 50  0000 L CNN
-F 1 "39k" V 8750 1550 50  0000 L CNN
+F 1 "10k" V 8750 1550 50  0000 L CNN
 F 2 "Resistors_SMD:R_0805" H 8700 1800 50  0001 C CNN
 F 3 "" H 8700 1800 50  0001 C CNN
@@
 P 8700 2050
 F 0 "R41" V 8750 2200 50  0000 L CNN
-F 1 "39k" V 8750 1800 50  0000 L CNN
+F 1 "10k" V 8750 1800 50  0000 L CNN
 F 2 "Resistors_SMD:R_0805" H 8700 2050 50  0001 C CNN
 F 3 "" H 8700 2050 50  0001 C CNN
@@
 P 8700 2300
 F 0 "R42" V 8750 2450 50  0000 L CNN
-F 1 "39k" V 8750 2050 50  0000 L CNN
+F 1 "10k" V 8750 2050 50  0000 L CNN
 F 2 "Resistors_SMD:R_0805" H 8700 2300 50  0001 C CNN
 F 3 "" H 8700 2300 50  0001 C CNN
@@
 P 8700 2550
 F 0 "R43" V 8750 2700 50  0000 L CNN
-F 1 "39k" V 8750 2300 50  0000 L CNN
+F 1 "10k" V 8750 2300 50  0000 L CNN
 F 2 "Resistors_SMD:R_0805" H 8700 2550 50  0001 C CNN
 F 3 "" H 8700 2550 50  0001 C CNN
@@
 P 8700 2800
 F 0 "R44" V 8750 2950 50  0000 L CNN
-F 1 "39k" V 8750 2550 50  0000 L CNN
+F 1 "10k" V 8750 2550 50  0000 L CNN
 F 2 "Resistors_SMD:R_0805" H 8700 2800 50  0001 C CNN
 F 3 "" H 8700 2800 50  0001 C CNN
@@
 P 8700 3050
 F 0 "R45" V 8750 3200 50  0000 L CNN
-F 1 "39k" V 8750 2800 50  0000 L CNN
+F 1 "10k" V 8750 2800 50  0000 L CNN
 F 2 "Resistors_SMD:R_0805" H 8700 3050 50  0001 C CNN
 F 3 "" H 8700 3050 50  0001 C CNN
@@
 P 8700 3300
 F 0 "R46" V 8750 3450 50  0000 L CNN
-F 1 "39k" V 8750 3050 50  0000 L CNN
+F 1 "10k" V 8750 3050 50  0000 L CNN
 F 2 "Resistors_SMD:R_0805" H 8700 3300 50  0001 C CNN
 F 3 "" H 8700 3300 50  0001 C CNN
@@
 	6850 3300 8600 3300
 Wire Wire Line
-	8800 1550 9100 1550
-Wire Wire Line
-	9100 1350 9100 3300
+	8800 1550 9800 1550
 Wire Wire Line
 	9100 3300 8800 3300
 Wire Wire Line
-	8800 3050 9100 3050
+	9100 3050 8800 3050
 Connection ~ 9100 3050
 Wire Wire Line
@@
 Connection ~ 9100 1800
 Wire Wire Line
-	8800 2050 9100 2050
+	9100 2050 8800 2050
 Connection ~ 9100 2050
 Wire Wire Line
-	8800 2300 9100 2300
+	9100 2300 8800 2300
 Connection ~ 9100 2300
 Wire Wire Line
-	8800 2550 9100 2550
+	9100 2550 8800 2550
 Connection ~ 9100 2550
 Wire Wire Line
-	8800 2800 9100 2800
+	9100 2800 8800 2800
 Connection ~ 9100 2800
 Connection ~ 9100 1550
@@
 L +3V3 #PWR053
 U 1 1 5966462B
-P 9300 3450
-F 0 "#PWR053" H 9300 3300 50  0001 C CNN
-F 1 "+3V3" H 9300 3590 50  0000 C CNN
-F 2 "" H 9300 3450 50  0001 C CNN
-F 3 "" H 9300 3450 50  0001 C CNN
-	1    9300 3450
-	1    0    0    -1
-$EndComp
-Wire Wire Line
-	9300 3450 9300 3500
-Wire Wire Line
-	5350 1350 9400 1350
-Wire Wire Line
-	4450 1700 5350 1700
-Wire Wire Line
-	5350 1700 5350 1350
-Connection ~ 4450 1700
+P 9800 1400
+F 0 "#PWR053" H 9800 1250 50  0001 C CNN
+F 1 "+3V3" H 9800 1540 50  0000 C CNN
+F 2 "" H 9800 1400 50  0001 C CNN
+F 3 "" H 9800 1400 50  0001 C CNN
+	1    9800 1400
+	1    0    0    -1
+$EndComp
+Wire Wire Line
+	9300 2100 9300 3500
 Wire Wire Line
 	4450 2000 4450 3950
@@
 L C_Small C16
 U 1 1 59A632A4
-P 9400 1550
-F 0 "C16" H 9500 1550 50  0000 L CNN
-F 1 "0,1uF 50V" H 9500 1450 50  0000 L CNN
-F 2 "Capacitors_SMD:C_0805" H 9400 1550 50  0001 C CNN
-F 3 "" H 9400 1550 50  0001 C CNN
-	1    9400 1550
+P 9800 2450
+F 0 "C16" H 9900 2450 50  0000 L CNN
+F 1 "0,1uF 50V" H 9900 2350 50  0000 L CNN
+F 2 "Capacitors_SMD:C_0805" H 9800 2450 50  0001 C CNN
+F 3 "" H 9800 2450 50  0001 C CNN
+	1    9800 2450
 	1    0    0    -1
 $EndComp
@@
 L Earth #PWR055
 U 1 1 59A63418
-P 9400 1750
-F 0 "#PWR055" H 9400 1500 50  0001 C CNN
-F 1 "Earth" H 9400 1600 50  0001 C CNN
-F 2 "" H 9400 1750 50  0001 C CNN
-F 3 "" H 9400 1750 50  0001 C CNN
-	1    9400 1750
-	1    0    0    -1
-$EndComp
-Wire Wire Line
-	9400 1350 9400 1450
-Connection ~ 9100 1350
-Wire Wire Line
-	9400 1650 9400 1750
+P 9800 2650
+F 0 "#PWR055" H 9800 2400 50  0001 C CNN
+F 1 "Earth" H 9800 2500 50  0001 C CNN
+F 2 "" H 9800 2650 50  0001 C CNN
+F 3 "" H 9800 2650 50  0001 C CNN
+	1    9800 2650
+	1    0    0    -1
+$EndComp
+Wire Wire Line
+	9800 2550 9800 2650
 Text GLabel 3350 4550 0    60   Input ~ 0
 3VA
@@
 NoConn ~ 4450 6400
 NoConn ~ 4450 6500
+Wire Wire Line
+	9100 1550 9100 3300
+Wire Wire Line
+	9800 1400 9800 2350
+Connection ~ 9800 1550
+Wire Wire Line
+	9300 2100 9800 2100
+Connection ~ 9800 2100
 $EndSCHEMATC
