File: Titan67j60/Titan67j60_NonSafety.sch (KiCad schematic (older format))
At the start: 68 parts, among them J19 CONN_01X03, J20 CONN_01X03, J21 CONN_01X03, J22 CONN_01X04, J23 CONN_01X03, J24 CONN_01X03, J25 CONN_01X03, J26 CONN_01X01, J27 CONN_01X03, J28 CONN_01X03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

Commit message: FirstProbe - мигает в локалке (XC8), SecondProbe - собирает TCP стек с HTTP2 (C18), FhirdProbe - пробуем с нуля писать без TCP стека (C18) TitanNonSafety - для ATtiny20 на высоковольтной стороне
Parts:
- C21: value 10,0 -> 22,0
- D10: value BZX84-C5V1 -> BZX84-C5V6
- R56, R60: value 240k -> 91k
- R73: value 75k -> 100k
- R74: value 130k -> 100k
- RV1: footprint Varistors:RV_Disc_D7_W4.3_P5 -> (none)
Connections:
- net ATplus: no longer U13.3 (EN)
- net ComOpto+: now also U12.6 ((PCINT7/SCL/SCK/T1/ICP1/OC0B/ADC7)PA7); no longer U12.9 ((PCINT4/ADC4)PA4)
- net at U12.13 ((PCINT0/ADC0)PA0): now also U13.3 (EN)
- no-connect marks 6 -> 5
Changed lines of the file:
@@
 P 2500 1900
 F 0 "R56" V 2300 1750 50  0000 L CNN
-F 1 "240k" V 2400 1750 50  0000 L CNN
+F 1 "91k" V 2400 1750 50  0000 L CNN
 F 2 "Resistors_SMD:R_1206" H 2500 1900 50  0001 C CNN
 F 3 "" H 2500 1900 50  0001 C CNN
@@
 P 8750 2300
 F 0 "C21" H 8760 2370 50  0000 L CNN
-F 1 "10,0" H 8760 2220 50  0000 L CNN
+F 1 "22,0" H 8760 2220 50  0000 L CNN
 F 2 "Capacitors_SMD:C_0805" H 8750 2300 50  0001 C CNN
 F 3 "" H 8750 2300 50  0001 C CNN
@@
 P 2800 1900
 F 0 "R60" V 2600 1750 50  0000 L CNN
-F 1 "240k" V 2700 1750 50  0000 L CNN
+F 1 "91k" V 2700 1750 50  0000 L CNN
 F 2 "Resistors_SMD:R_1206" H 2800 1900 50  0001 C CNN
 F 3 "" H 2800 1900 50  0001 C CNN
@@
 P 9050 2250
 F 0 "D10" V 8900 2150 50  0000 C CNN
-F 1 "BZX84-C5V1" H 9350 2350 50  0000 C CNN
+F 1 "BZX84-C5V6" H 9350 2350 50  0000 C CNN
 F 2 "Diodes_SMD:D_SOT-23_ANK" H 9050 2250 50  0001 C CNN
 F 3 "" H 9050 2250 50  0001 C CNN
@@
 F 0 "RV1" V 2625 1050 50  0000 C CNN
 F 1 "Varistor" V 2375 1050 50  0000 C CNN
-F 2 "Varistors:RV_Disc_D7_W4.3_P5" V 2430 1050 50  0001 C CNN
+F 2 "" V 2430 1050 50  0001 C CNN
 F 3 "" H 2500 1050 50  0001 C CNN
 	1    2500 1050
@@
 P 7900 5450
 F 0 "R73" H 8000 5400 50  0000 L CNN
-F 1 "75k" H 8000 5500 50  0000 L CNN
+F 1 "100k" H 8000 5500 50  0000 L CNN
 F 2 "Resistors_SMD:R_0603" H 7900 5450 50  0001 C CNN
 F 3 "" H 7900 5450 50  0001 C CNN
@@
 P 8000 4550
 F 0 "R74" H 8150 4550 50  0000 L CNN
-F 1 "130k" H 8100 4650 50  0000 L CNN
+F 1 "100k" H 8100 4650 50  0000 L CNN
 F 2 "Resistors_SMD:R_1206" H 8000 4550 50  0001 C CNN
 F 3 "" H 8000 4550 50  0001 C CNN
@@
 Wire Wire Line
 	8250 3400 8350 3400
-Wire Wire Line
-	8250 1700 8250 3800
 Connection ~ 8250 1700
-Wire Wire Line
-	7050 3800 8350 3800
 Connection ~ 8250 3400
 Wire Wire Line
@@
 Connection ~ 7900 1700
 Wire Wire Line
-	5400 2100 4000 2100
-Wire Wire Line
 	3050 1500 3050 1900
 Wire Wire Line
@@
 Wire Wire Line
 	4000 2500 3900 2500
-Connection ~ 4000 2100
 Wire Wire Line
 	7800 3250 7900 3250
@@
 Wire Wire Line
 	7050 5250 8400 5250
-Wire Wire Line
-	7050 5250 7050 3800
-Connection ~ 8250 3800
 Wire Wire Line
 	7900 5350 7900 5250
@@
 	0    -1   -1   0
 $EndComp
-NoConn ~ 5400 2400
 Wire Wire Line
 	4650 3200 4650 2700
 Wire Wire Line
 	4650 2600 5400 2600
-NoConn ~ 5400 1700
 Wire Wire Line
 	4650 2600 4650 1500
@@
 	-1   0    0    -1
 $EndComp
+Wire Wire Line
+	5400 2400 4000 2400
+Connection ~ 4000 2400
+Wire Wire Line
+	8250 1700 8250 4000
+Wire Wire Line
+	8250 4000 7050 4000
+Wire Wire Line
+	7050 4000 7050 5250
+Wire Wire Line
+	5400 1700 4750 1700
+Wire Wire Line
+	4750 1700 4750 3800
+Wire Wire Line
+	4750 3800 8350 3800
+NoConn ~ 5400 2100
 $EndSCHEMATC

Commit message: Работает минимальный набор до прикручивания TCP IP
Signed-off-by: Lehman3065 <lehman3065@gmail.com>
Parts:
- R77: value 100k -> 200k
Changed lines of the file:
@@
 P 8050 5800
 F 0 "R77" H 7800 5850 50  0000 L CNN
-F 1 "100k" H 7800 5750 50  0000 L CNN
+F 1 "200k" H 7800 5750 50  0000 L CNN
 F 2 "Resistors_SMD:R_0603" H 8050 5800 50  0001 C CNN
 F 3 "" H 8050 5800 50  0001 C CNN
