File: Titan67j60/Titan67j60_PowerSupply.sch (KiCad schematic (older format))
At the start: 40 parts, among them T2 EF20 Core, U14 Viper37LD, U15 PC817, U16 TL431IDBZR

Commit message: FirstProbe - мигает в локалке (XC8), SecondProbe - собирает TCP стек с HTTP2 (C18), FhirdProbe - пробуем с нуля писать без TCP стека (C18) TitanNonSafety - для ATtiny20 на высоковольтной стороне
Parts:
- RV2: footprint Varistors:RV_Disc_D7_W3.4_P5 -> (none)
Changed lines of the file:
@@
 F 0 "RV2" V 3225 4500 50  0000 C CNN
 F 1 "471" V 2975 4500 50  0000 C CNN
-F 2 "Varistors:RV_Disc_D7_W3.4_P5" V 3030 4500 50  0001 C CNN
+F 2 "" V 3030 4500 50  0001 C CNN
 F 3 "" H 3100 4500 50  0001 C CNN
 	1    3100 4500

Commit message: Работает минимальный набор до прикручивания TCP IP
Signed-off-by: Lehman3065 <lehman3065@gmail.com>
Parts:
- C31: value 56n -> 0,15
- R85: value 75k -> 200k
- R86: value 18k -> 39k
Changed lines of the file:
@@
 P 6050 3300
 F 0 "R85" H 6080 3320 50  0000 L CNN
-F 1 "75k" H 5800 3350 50  0000 L CNN
+F 1 "200k" H 5800 3350 50  0000 L CNN
 F 2 "Resistors_SMD:R_0805" H 6050 3300 50  0001 C CNN
 F 3 "" H 6050 3300 50  0001 C CNN
@@
 P 6050 3700
 F 0 "R86" H 6080 3720 50  0000 L CNN
-F 1 "18k" H 5850 3700 50  0000 L CNN
+F 1 "39k" H 5850 3700 50  0000 L CNN
 F 2 "Resistors_SMD:R_0805" H 6050 3700 50  0001 C CNN
 F 3 "" H 6050 3700 50  0001 C CNN
@@
 P 3900 3900
 F 0 "C31" H 3910 3970 50  0000 L CNN
-F 1 "56n" H 3910 3820 50  0000 L CNN
+F 1 "0,15" H 3910 3820 50  0000 L CNN
 F 2 "Capacitors_SMD:C_0805" H 3900 3900 50  0001 C CNN
 F 3 "" H 3900 3900 50  0001 C CNN
